Commit message: 修改了一些bug

File: unitree_hardware_interface/description/quadruped.urdf.xacro (robot description, xacro)
@@ -8,4 +8,9 @@
       <child link="motor_${index}_link"/>
       <limit effort="50" velocity="30" lower="-12.56" upper="12.56"/>
+    </joint>
+    <link name="motor_${index}_link"/>
+  </xacro:macro>
+  <xacro:macro name="ros_joint" params="index">
+    <joint name="joint_${index}">
       <command_interface name="position"/>
       <command_interface name="velocity"/>
@@ -15,26 +20,21 @@
       <state_interface name="effort"/>
     </joint>
-    <link name="motor_${index}_link"/>
   </xacro:macro>
   <link name="base_link"/>
-  <xacro:macro name="all_motors">
-    <xacro:motor_joint index="0"/>
-    <xacro:motor_joint index="1"/>
-    <xacro:motor_joint index="2"/>
-    <xacro:motor_joint index="3"/>
-    <xacro:motor_joint index="4"/>
-    <xacro:motor_joint index="5"/>
-    <xacro:motor_joint index="6"/>
-    <xacro:motor_joint index="7"/>
-    <xacro:motor_joint index="8"/>
-    <xacro:motor_joint index="9"/>
-    <xacro:motor_joint index="10"/>
-    <xacro:motor_joint index="11"/>
-  </xacro:macro>
-  <xacro:all_motors/>
+  <xacro:motor_joint index="0"/>
+  <xacro:motor_joint index="1"/>
+  <xacro:motor_joint index="2"/>
+  <xacro:motor_joint index="3"/>
+  <xacro:motor_joint index="4"/>
+  <xacro:motor_joint index="5"/>
+  <xacro:motor_joint index="6"/>
+  <xacro:motor_joint index="7"/>
+  <xacro:motor_joint index="8"/>
+  <xacro:motor_joint index="9"/>
+  <xacro:motor_joint index="10"/>
+  <xacro:motor_joint index="11"/>
   <ros2_control name="UnitreeHardwareInterface" type="system">
     <hardware>
       <plugin>unitree_hardware_interface/UnitreeHardwareInterface</plugin>
-      <!-- Default port mapping: USB0→motors 0-2, USB1→3-5, USB2→6-8, USB3→9-11 -->
       <param name="port_0">/dev/ttyUSB0:0</param>
       <param name="port_1">/dev/ttyUSB1:3</param>
@@ -46,4 +46,16 @@
       <param name="timeout_us">20000</param>
     </hardware>
+    <xacro:ros_joint index="0"/>
+    <xacro:ros_joint index="1"/>
+    <xacro:ros_joint index="2"/>
+    <xacro:ros_joint index="3"/>
+    <xacro:ros_joint index="4"/>
+    <xacro:ros_joint index="5"/>
+    <xacro:ros_joint index="6"/>
+    <xacro:ros_joint index="7"/>
+    <xacro:ros_joint index="8"/>
+    <xacro:ros_joint index="9"/>
+    <xacro:ros_joint index="10"/>
+    <xacro:ros_joint index="11"/>
   </ros2_control>
 </robot>
